File: placa-expansion/placa-expansion.kicad_pcb (KiCad board)
At the start: 2 copper layers, 70 x 114.2 mm, 24 parts, among them J1 PBD-26, P1 BATT, P2 CONN_3PI, P3 PWR_HUB, P4 PWR_3pi, P5 CONN_4, P6 CONN_4, P7 CONN_4, P8 CONN_4, U1 PTN78020

Commit message: modifico un par de pistas
Routing:
- net /TX_3pi: track 106.0 -> 110.8 mm
Other:
- net class Default: clearance 0.254 -> 0.508; trace_width 0.381 -> 0.762
- rule trace_clearance: 0.254 -> 0.508
Changed lines of the file:
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@@
     (links 59)
     (no_connects 0)
-    (area 159.881999 91.149999 230.100001 205.600001)
+    (area 159.3084 90.6 231.04942 206.0396)
     (thickness 1.6)
     (drawings 9)
-    (tracks 287)
+    (tracks 291)
     (zones 0)
     (modules 24)
@@
   )
   (setup
-    (last_trace_width 0.381)
+    (last_trace_width 0.762)
     (user_trace_width 0.3048)
     (user_trace_width 0.4064)
     (user_trace_width 0.508)
-    (trace_clearance 0.254)
+    (trace_clearance 0.508)
     (zone_clearance 0.381)
     (zone_45_only no)
@@
   (net 42 N-000008)
   (net_class Default "This is the default net class."
-    (clearance 0.254)
-    (trace_width 0.381)
+    (clearance 0.508)
+    (trace_width 0.762)
     (via_dia 2)
     (via_drill 0.7)
@@
   (segment (start 168.516 173.016) (end 165.252 173.016) (width 0.762) (layer B.Cu) (net 14))
   (segment (start 173.66318 178.16318) (end 173 177.5) (width 0.381) (layer B.Cu) (net 14))
+  (segment (start 182.83188 185.1) (end 182.83188 189.23188) (width 0.762) (layer B.Cu) (net 15))
+  (segment (start 182.83188 189.23188) (end 183 189.4) (width 0.762) (layer B.Cu) (net 15))
   (segment (start 175 133.2) (end 174.6 133.6) (width 0.762) (layer F.Cu) (net 15))
   (segment (start 180.5 189.4) (end 183 189.4) (width 0.762) (layer F.Cu) (net 15))
   (segment (start 174.6 183.5) (end 180.5 189.4) (width 0.762) (layer F.Cu) (net 15))
   (segment (start 174.6 133.6) (end 174.6 183.5) (width 0.762) (layer F.Cu) (net 15))
-  (segment (start 182.83188 182.05954) (end 182.83188 189.23188) (width 0.381) (layer B.Cu) (net 15))
+  (segment (start 182.83188 182.05954) (end 182.83188 185.1) (width 0.381) (layer B.Cu) (net 15))
   (segment (start 182.83188 189.23188) (end 183 189.4) (width 0.381) (layer B.Cu) (net 15))
   (segment (start 183 189.5) (end 183 189.3) (width 0.762) (layer B.Cu) (net 15))
@@
   (via (at 169.4 185.5) (size 2) (layers F.Cu B.Cu) (net 16))
   (segment (start 169.4 185.5) (end 169.4 165.2) (width 0.762) (layer F.Cu) (net 16))
-  (segment (start 161.316 185.716) (end 162.712 185.716) (width 0.381) (layer B.Cu) (net 16) (status 800000))
+  (segment (start 161.316 185.716) (end 162.712 185.716) (width 0.381) (layer B.Cu) (net 16))
   (segment (start 160.8 185.2) (end 161.316 185.716) (width 0.381) (layer B.Cu) (net 16))
   (segment (start 170.4 185.5) (end 171.3 184.6) (width 0.762) (layer B.Cu) (net 16))
@@
   (segment (start 171.3 184.6) (end 175.14094 180.75906) (width 0.381) (layer B.Cu) (net 16))
   (segment (start 175.14094 180.75906) (end 177.13212 180.75906) (width 0.381) (layer B.Cu) (net 16))
+  (segment (start 180.3 183.3) (end 180.3 186.7) (width 0.762) (layer B.Cu) (net 17))
+  (segment (start 180.3 186.7) (end 176.9 190.1) (width 0.762) (layer B.Cu) (net 17))
   (segment (start 182.83188 180.75906) (end 181.14094 180.75906) (width 0.381) (layer B.Cu) (net 17))
   (segment (start 180.3 186.7) (end 176.9 190.1) (width 0.381) (layer B.Cu) (net 17))
-  (segment (start 180.3 181.6) (end 180.3 186.7) (width 0.381) (layer B.Cu) (net 17))
+  (segment (start 180.3 181.6) (end 180.3 183.3) (width 0.381) (layer B.Cu) (net 17))
   (segment (start 181.14094 180.75906) (end 180.3 181.6) (width 0.381) (layer B.Cu) (net 17))
   (via (at 176.9 190.1) (size 2) (layers F.Cu B.Cu) (net 17))
@@
   (via (at 191.9 119.6) (size 2) (layers F.Cu B.Cu) (net 17))
   (segment (start 191.942 119.642) (end 191.9 119.6) (width 0.762) (layer B.Cu) (net 17))
-  (segment (start 177.13212 182.05954) (end 176.74046 182.05954) (width 0.381) (layer B.Cu) (net 18) (status C00000))
-  (segment (start 176.74046 182.05954) (end 174 184.8) (width 0.381) (layer B.Cu) (net 18) (status 400000))
+  (segment (start 177.13212 182.05954) (end 176.74046 182.05954) (width 0.381) (layer B.Cu) (net 18))
+  (segment (start 176.74046 182.05954) (end 174 184.8) (width 0.381) (layer B.Cu) (net 18))
   (segment (start 161.7 198.5) (end 168.5 198.5) (width 0.762) (layer F.Cu) (net 18))
   (segment (start 160.756 188.256) (end 160.7 188.2) (width 0.381) (layer B.Cu) (net 18))
@@
   (segment (start 160.8 188.3) (end 160.8 197.6) (width 0.381) (layer F.Cu) (net 18))
   (segment (start 160.8 197.6) (end 161.7 198.5) (width 0.381) (layer F.Cu) (net 18))
-  (segment (start 160.756 188.256) (end 162.712 188.256) (width 0.381) (layer B.Cu) (net 18) (status 800000))
+  (segment (start 160.756 188.256) (end 162.712 188.256) (width 0.381) (layer B.Cu) (net 18))
   (segment (start 169.6 189.2) (end 174 184.8) (width 0.762) (layer B.Cu) (net 18))
   (via (at 169.6 189.2) (size 2) (layers F.Cu B.Cu) (net 18))

Commit message: subo archivos de fabricacion para el LCI, capas: drill, soldermask y copper
Routing:
- net /AD6: track 105.2 -> 116.1 mm
- net GND: track 2.54 -> 12.6 mm, vias 0 -> 1
- net /PC6: track 270.9 -> 280.6 mm
- net /RX_3pi: track 92.6 -> 97.1 mm
- net /AD7: track 105.2 -> 107.9 mm
- net /Echo4: track 136.1 -> 138.6 mm
- net N-0000042: track 24.5 -> 22.6 mm
- net +5V: track 240.7 -> 242.5 mm
Other:
- net class Default: via_dia 2 -> 1
